Commit message: re-factor base controller to use ros-control

File: src/smart_description/urdf/smart_base.urdf.xacro (robot description, xacro)
@@ -1,5 +1,5 @@
 <?xml version="1.0"?>
 <robot xmlns:xacro="http://ros.org/wiki/xacro">
-  <xacro:include filename="$(find smart_description)/urdf/smart_wheel_suspension.urdf.xacro" />
+  <xacro:include filename="$(find smart_description)/urdf/smart_wheel_steering.urdf.xacro" />
   <xacro:include filename="$(find smart_description)/urdf/smart_wheel.urdf.xacro" />
   <xacro:include filename="$(find smart_description)/urdf/smart_camera_mast.urdf.xacro" />
@@ -21,10 +21,10 @@
       </collision>
     </link>
-    <xacro:smart_wheel_suspension parent="base_link" prefix="front" suffix="left" reflect_x="1" reflect_y="1" mount_joint_type="revolute" />
-    <xacro:smart_wheel_suspension parent="base_link" prefix="front" suffix="right" reflect_x="1" reflect_y="-1" mount_joint_type="revolute" />
-    <xacro:smart_wheel_suspension parent="base_link" prefix="middle" suffix="left" reflect_x="0" reflect_y="1" mount_joint_type="revolute" />
-    <xacro:smart_wheel_suspension parent="base_link" prefix="middle" suffix="right" reflect_x="0" reflect_y="-1" mount_joint_type="revolute" />
-    <xacro:smart_wheel_suspension parent="base_link" prefix="rear" suffix="left" reflect_x="-1" reflect_y="1" mount_joint_type="revolute" />
-    <xacro:smart_wheel_suspension parent="base_link" prefix="rear" suffix="right" reflect_x="-1" reflect_y="-1" mount_joint_type="revolute" />
+    <xacro:smart_wheel_steering parent="base_link" prefix="front" suffix="left" reflect_x="1" reflect_y="1" mount_joint_type="revolute" />
+    <xacro:smart_wheel_steering parent="base_link" prefix="front" suffix="right" reflect_x="1" reflect_y="-1" mount_joint_type="revolute" />
+    <xacro:smart_wheel_steering parent="base_link" prefix="middle" suffix="left" reflect_x="0" reflect_y="1" mount_joint_type="revolute" />
+    <xacro:smart_wheel_steering parent="base_link" prefix="middle" suffix="right" reflect_x="0" reflect_y="-1" mount_joint_type="revolute" />
+    <xacro:smart_wheel_steering parent="base_link" prefix="rear" suffix="left" reflect_x="-1" reflect_y="1" mount_joint_type="revolute" />
+    <xacro:smart_wheel_steering parent="base_link" prefix="rear" suffix="right" reflect_x="-1" reflect_y="-1" mount_joint_type="revolute" />
     <xacro:smart_wheel parent="motor_link" prefix="front" suffix="left" wheel_joint_type="${wheel_joint_type}" />
     <xacro:smart_wheel parent="motor_link" prefix="front" suffix="right" wheel_joint_type="${wheel_joint_type}" />

File: src/smart_description/urdf/smart_parameters.urdf.xacro (robot description, xacro)
@@ -3,7 +3,7 @@
   <!-- Properties (Constants) -->
   <xacro:property name="M_PI" value="3.1415926535897931" />
-  <xacro:property name="wheel_suspension_offset_x" value="0.15" />
-  <xacro:property name="wheel_suspension_offset_y" value="0.1435" />
-  <xacro:property name="wheel_suspension_offset_z" value="0" />
+  <xacro:property name="wheel_steering_offset_x" value="0.15" />
+  <xacro:property name="wheel_steering_offset_y" value="0.1435" />
+  <xacro:property name="wheel_steering_offset_z" value="0" />
   <xacro:property name="wheel_radius" value="0.035" />
   <xacro:property name="wheel_size_y" value="0.035" />

File: src/smart_description/urdf/smart_wheel_steering.urdf.xacro (robot description, xacro)
@@ -2,13 +2,13 @@
 <robot xmlns:xacro="http://ros.org/wiki/xacro">
   <xacro:include filename="$(find smart_description)/urdf/smart_parameters.urdf.xacro" />
-  <xacro:macro name="smart_wheel_suspension" params="parent prefix suffix reflect_x reflect_y mount_joint_type">
-    <joint name="${prefix}_${suffix}_wheel_suspension_joint" type="${mount_joint_type}">
-      <origin xyz="${wheel_suspension_offset_x * reflect_x} ${wheel_suspension_offset_y * reflect_y} ${wheel_suspension_offset_z}" rpy="0 0 0" />
+  <xacro:macro name="smart_wheel_steering" params="parent prefix suffix reflect_x reflect_y mount_joint_type">
+    <joint name="${prefix}_${suffix}_wheel_steering_joint" type="${mount_joint_type}">
+      <origin xyz="${wheel_steering_offset_x * reflect_x} ${wheel_steering_offset_y * reflect_y} ${wheel_steering_offset_z}" rpy="0 0 0" />
       <parent link="${parent}" />
-      <child link="${prefix}_${suffix}_wheel_suspension_link" />
+      <child link="${prefix}_${suffix}_wheel_steering_link" />
       <axis xyz="0 0 1" />
       <limit lower="${-M_PI}" upper="${M_PI}" effort="100" velocity="100" />
     </joint>
-    <link name="${prefix}_${suffix}_wheel_suspension_link">
+    <link name="${prefix}_${suffix}_wheel_steering_link">
       <inertial>
         <mass value="0.01" />
@@ -21,5 +21,5 @@
         <origin xyz="0.0 0.0 0.0" rpy="0 0 ${M_PI * ((reflect_y / 2) + 0.5)}" />
         <geometry>
-          <mesh filename="package://smart_description/meshes/smart_wheel_suspension.dae" scale=" 0.01  0.01  0.01" />
+          <mesh filename="package://smart_description/meshes/smart_wheel_steering.dae" scale=" 0.01  0.01  0.01" />
         </geometry>
       </visual>
@@ -27,5 +27,5 @@
         <origin xyz="0.0 0.0 0.0" rpy="0 0 ${M_PI * ((reflect_y / 2) + 0.5)}" />
         <geometry>
-          <mesh filename="package://smart_description/meshes/smart_wheel_suspension.stl" scale=" 0.01  0.01  0.01" />
+          <mesh filename="package://smart_description/meshes/smart_wheel_steering.stl" scale=" 0.01  0.01  0.01" />
         </geometry>
       </collision>
@@ -33,5 +33,5 @@
    <joint name="${prefix}_${suffix}_motor_joint" type="fixed">
       <origin xyz="0 0 ${wheel_offset_z}" rpy="0 0 0" />
-      <parent link="${prefix}_${suffix}_wheel_suspension_link" />
+      <parent link="${prefix}_${suffix}_wheel_steering_link" />
       <child link="${prefix}_${suffix}_motor_link" />
     </joint>

Commit message: replaced base mesh by a simplified model for debugging

File: src/smart_description/urdf/smart_base.urdf.xacro (robot description, xacro)
@@ -11,5 +11,6 @@
         <origin xyz="0.0 0.0 0.0" rpy="0 0 0" />
         <geometry>
-          <mesh filename="package://smart_description/meshes/smart_base.dae" scale=" 0.01  0.01  0.01"/>
+          <!-- mesh filename="package://smart_description/meshes/smart_base.dae" scale=" 0.01  0.01  0.01"/ -->
+          <cylinder radius="0.1" length="0.1" />
         </geometry>
       </visual>
@@ -17,5 +18,6 @@
         <origin xyz="0.0 0.0 0.0" rpy="0 0 0" />
         <geometry>
-          <mesh filename="package://smart_description/meshes/smart_base.stl" scale=" 0.01  0.01  0.01"/>
+          <!-- mesh filename="package://smart_description/meshes/smart_base.stl" scale=" 0.01  0.01  0.01"/ -->
+          <cylinder radius="0.1" length="0.1" />
         </geometry>
       </collision>

Commit message: enabled ros melodic compatibility removed ros_control interface added smart_gazebo_plugin

File: src/smart_description/urdf/smart_base.urdf.xacro (robot description, xacro)
@@ -11,6 +11,5 @@
         <origin xyz="0.0 0.0 0.0" rpy="0 0 0" />
         <geometry>
-          <!-- mesh filename="package://smart_description/meshes/smart_base.dae" scale=" 0.01  0.01  0.01"/ -->
-          <cylinder radius="0.1" length="0.1" />
+          <mesh filename="package://smart_description/meshes/smart_base.dae" scale=" 0.01  0.01  0.01"/>
         </geometry>
       </visual>
@@ -18,6 +17,5 @@
         <origin xyz="0.0 0.0 0.0" rpy="0 0 0" />
         <geometry>
-          <!-- mesh filename="package://smart_description/meshes/smart_base.stl" scale=" 0.01  0.01  0.01"/ -->
-          <cylinder radius="0.1" length="0.1" />
+          <mesh filename="package://smart_description/meshes/smart_base.stl" scale=" 0.01  0.01  0.01"/>
         </geometry>
       </collision>

File: src/smart_gazebo/urdf/smart_gazebo.urdf.xacro (robot description, xacro)
@@ -12,3 +12,5 @@
   <xacro:include filename="$(find smart_gazebo)/urdf/smart_materials.urdf.xacro" />
   <xacro:smart_materials/>
+  <xacro:include filename="$(find smart_gazebo)/urdf/smart_base_controllers.urdf.xacro" />
+  <xacro:smart_base_controllers/>
 </robot>

File: src/smart_gazebo/urdf/smart_materials.urdf.xacro (robot description, xacro)
@@ -1,5 +1,5 @@
 <?xml version="1.0"?>
 <robot xmlns:xacro="http://ros.org/wiki/xacro">
- <macro name="smart_materials">
+ <xacro:macro name="smart_materials">
   <!-- GAZEBO MATERIALS -->
   <gazebo reference="base_link">
@@ -63,4 +63,4 @@
     <material>Gazebo/Grey</material>
   </gazebo>
-</macro>
+</xacro:macro>
 </robot>
